File: Interface.kicad_sch (KiCad schematic)
At the start: 0 parts

Commit message: CIPOS circuit
Parts:
- added C31, C32, C33: C, symbol Device:C
- added R5, R6: R, symbol Device:R
- added U8: TCAN1042HGVDRBRQ1, DRB0008F, symbol TCAN1042HGVDRBRQ1:TCAN1042HGVDRBRQ1
Connections:
- new net: C31.1, R5.2, R6.1
- new net +3V3: C33.1, U8.5 (VIO)
- new net +5V: C32.1, U8.3 (VCC)
- new net CANH: R5.1, U8.7 (CANH)
- new net CANL: R6.2, U8.6 (CANL)
- new net CANRX: U8.4 (RXD)
- new net CANSTB: U8.8 (STB)
- new net CANTX: U8.1 (TXD)
- new net GND: C31.2, C32.2, C33.2, U8.2 (GND), U8.9 (PAD)
Other:
- note added: "CAN Transceiver"
- note added: "Data-Sheet"

Commit message: #
Parts:
- added J2, J3: Conn_01x02_Pin, symbol Connector:Conn_01x02_Pin
- added TP10, TP11, TP8, TP9: TestPoint, symbol Connector:TestPoint
- R5, R6: value R -> 60
Connections:
- net +3V3: now also J3.1 (Pin_1); no longer C33.1, U8.5 (VIO)
- net +5V: now also J2.1 (Pin_1); no longer C32.1, U8.3 (VCC)
- net CANH: now also TP8.1
- net CANL: now also TP9.1
- net CANRX: now also TP10.1
- net CANTX: now also TP11.1
- new net VCC: C32.1, J2.2 (Pin_2), U8.3 (VCC)
- new net VIO: C33.1, J3.2 (Pin_2), U8.5 (VIO)

Commit message: #
Other:
- moved on the sheet: C31, C32, C33, J2, J3, R5, R6, TP10, TP11, TP8, TP9, U8

Commit message: #
Parts:
- C19: renamed from C33; value C -> 0.1u
- C20: renamed from C32; value C -> 0.1u
- C21: renamed from C31; value C -> 0.1u; now not fitted
- U8: footprint DRB0008F -> Footprint:DRB0008F
- renumbered R5 to R30, R6 to R31
Connections:
- net +3V3 renamed +3.3V
Other:
- moved on the sheet: C19, C20, J2, J3, R30, R31, TP10, TP11, TP8, TP9, U8
