File: Inverter.kicad_sch (KiCad schematic)
At the start: 0 parts

Commit message: CIPOS circuit
Other:
- added sheet Inverter_PowerStage (Inverter_PowerStage.kicad_sch)
Changed lines of the file:
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@@
+	)
+	(sheet
+		(at 34.544 76.454)
+		(size 51.816 27.94)
+		(exclude_from_sim no)
+		(in_bom yes)
+		(on_board yes)
+		(dnp no)
+		(fields_autoplaced yes)
+		(stroke
+			(width 0.1524)
+			(type solid)
+		)
+		(fill
+			(color 0 0 0 0)
+		)
+		(property "Sheetname" "Inverter_PowerStage"
+			(at 34.544 75.7424 0)
+			(show_name no)
+			(do_not_autoplace no)
+			(effects
+				(font
+					(size 1.27 1.27)
+				)
+				(justify left bottom)
+			)
+		)
+		(property "Sheetfile" "Inverter_PowerStage.kicad_sch"
+			(at 34.544 104.9786 0)
+			(show_name no)
+			(do_not_autoplace no)
+			(effects
+				(font
+					(size 1.27 1.27)
+				)
+				(justify left top)
+			)
+		)
+		(instances
+			(project "Inverter"
+				(path "/557dbdfe-f200-4573-9e2e-e58e9c4cef92"
+					(page "6")
+				)
+			)
+		)
 	)
 	(sheet

Commit message: #
Other:
- added sheet MCU_comp (MCU_comp.kicad_sch)
- added sheet Ports (Ports.kicad_sch)
Changed lines of the file:
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@@
 	(generator_version "10.0")
 	(paper "A4")
+	(text_box "Power SW"
+		(exclude_from_sim no)
+		(at 36.068 30.734 0)
+		(size 47.752 30.734)
+		(margins 0.9525 0.9525 0.9525 0.9525)
+		(stroke
+			(width 0)
+			(type solid)
+		)
+		(fill
+			(type none)
+		)
+		(effects
+			(font
+				(size 2.54 2.54)
+				(thickness 0.3175)
+			)
+		)
+	)
 	(text_box "TMS570LS0714"
 		(exclude_from_sim no)
-		(at 95.25 30.48 0)
+		(at 95.25 31.496 0)
 		(size 46.99 29.21)
 		(margins 0.9525 0.9525 0.9525 0.9525)
@@
 		(effects
 			(font
-				(size 1.27 1.27)
-			)
-			(justify left top)
+				(size 2.54 2.54)
+				(thickness 0.3175)
+			)
+		)
+	)
+	(text_box "MCU components (JTAG, Jumpers)"
+		(exclude_from_sim no)
+		(at 95.25 77.47 0)
+		(size 46.736 24.384)
+		(margins 0.9525 0.9525 0.9525 0.9525)
+		(stroke
+			(width 0)
+			(type solid)
+		)
+		(fill
+			(type none)
+		)
+		(effects
+			(font
+				(size 2.54 2.54)
+				(thickness 0.3175)
+			)
+		)
+	)
+	(text_box "Ports"
+		(exclude_from_sim no)
+		(at 151.892 76.962 0)
+		(size 42.164 25.654)
+		(margins 0.9525 0.9525 0.9525 0.9525)
+		(stroke
+			(width 0)
+			(type solid)
+		)
+		(fill
+			(type none)
+		)
+		(effects
+			(font
+				(size 2.54 2.54)
+				(thickness 0.3175)
+			)
+		)
+	)
+	(text_box "Sensors"
+		(exclude_from_sim no)
+		(at 153.416 31.496 0)
+		(size 39.37 28.956)
+		(margins 0.9525 0.9525 0.9525 0.9525)
+		(stroke
+			(width 0)
+			(type solid)
+		)
+		(fill
+			(type none)
+		)
+		(effects
+			(font
+				(size 2.54 2.54)
+				(thickness 0.3175)
+			)
 		)
 	)
@@
 	)
 	(sheet
+		(at 149.352 75.692)
+		(size 46.99 28.194)
+		(exclude_from_sim no)
+		(in_bom yes)
+		(on_board yes)
+		(dnp no)
+		(fields_autoplaced yes)
+		(stroke
+			(width 0.1524)
+			(type solid)
+		)
+		(fill
+			(color 0 0 0 0)
+		)
+		(property "Sheetname" "Ports"
+			(at 149.352 74.9804 0)
+			(show_name no)
+			(do_not_autoplace no)
+			(effects
+				(font
+					(size 1.27 1.27)
+				)
+				(justify left bottom)
+			)
+		)
+		(property "Sheetfile" "Ports.kicad_sch"
+			(at 149.352 104.4706 0)
+			(show_name no)
+			(do_not_autoplace no)
+			(effects
+				(font
+					(size 1.27 1.27)
+				)
+				(justify left top)
+			)
+		)
+		(instances
+			(project "Inverter"
+				(path "/557dbdfe-f200-4573-9e2e-e58e9c4cef92"
+					(page "8")
+				)
+			)
+		)
+	)
+	(sheet
 		(at 34.29 29.21)
 		(size 52.07 34.29)
@@
 				)
 			)
+		)
+	)
+	(sheet
+		(at 93.98 75.946)
+		(size 50.038 28.194)
+		(exclude_from_sim no)
+		(in_bom yes)
+		(on_board yes)
+		(dnp no)
+		(fields_autoplaced yes)
+		(stroke
+			(width 0.1524)
+			(type solid)
+		)
+		(fill
+			(color 0 0 0 0)
+		)
+		(property "Sheetname" "MCU_comp"
+			(at 93.98 75.2344 0)
+			(show_name no)
+			(do_not_autoplace no)
+			(effects
+				(font
+					(size 1.27 1.27)
+				)
+				(justify left bottom)
+			)
+		)
+		(property "Sheetfile" "MCU_comp.kicad_sch"
+			(at 93.98 104.7246 0)
+			(show_name no)
+			(do_not_autoplace no)
+			(effects
+				(font
+					(size 1.27 1.27)
+				)
+				(justify left top)
+			)
+		)
+		(instances
+			(project "Inverter"
+				(path "/557dbdfe-f200-4573-9e2e-e58e9c4cef92"
+					(page "7")
+				)
+			)
