File: power_sm.kicad_sch (KiCad schematic)
At the start: 37 parts, among them J1 Conn_01x02_Pin, J4 Conn_01x02_Pin, J5 Conn_01x02_Pin, J6 Conn_01x02_Pin, J7 Conn_01x02_Pin, J8 Conn_01x02_Pin, J9 Conn_01x02_Pin, U2 LM63460AASQRYFRQ1, U3 TPS78533QKVURQ1, U4 TLV70012QDDCRQ1

Commit message: CIPOS circuit
Parts:
- added C28, C30: 1uF, symbol Device:C
- added C29: 0.1uF, symbol Device:C
- added U7: REF35125QDBVRQ1, symbol Library:REF35125-Q1
Connections:
- net +3.3V: now also C29.1, U7.3 (EN), U7.4 (VIN)
- net GND: now also C28.2, C29.2, C30.1, U7.1 (GND), U7.2 (GND)
- new net: C30.2, U7.5 (NR)
- new net REFV: C28.1, U7.6 (VREF)
Other:
- note added: "+1.25V Vref"
- note added: "Data-Sheet"
- note added: "Ref for TLV6001"
- moved on the sheet: C1, C12, C13, C14, C15, C16, C17, C2, C3, C4, C5, C6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

Commit message: #
Parts:
- added C51: C, symbol Device:C
- added D10, D6, D7, D8, D9: LED, symbol Device:LED
- added FB5: FerriteBead, Inductor_SMD:L_0805_2012Metric_Pad1.05x1.20mm_HandSolder, symbol Device:FerriteBead
- added R20, R21, R22, R23, R24: R, symbol Device:R
Connections:
- net +15V: now also D9.2 (A)
- net +1V2: now also D8.2 (A)
- net +3.3V: now also D7.2 (A)
- net +5V: now also D6.2 (A)
- net +5VA: now also D10.2 (A)
- net GND: now also R20.2, R21.2, R22.2
- net GND1: now also R23.2, R24.2
- net REFV: now also FB5.2; no longer C28.1, U7.6 (VREF)
- new net: D8.1 (K), R22.1
- new net: C28.1, FB5.1, U7.6 (VREF)
- new net: D9.1 (K), R23.1
- new net: D10.1 (K), R24.1
- new net: D6.1 (K), R20.1
- new net: D7.1 (K), R21.1
Other:
- note added: "Supply for sensors"
- moved on the sheet: C28, C29, C30, U7

Commit message: #
Parts:
- removed C28, C30: 1uF, symbol Device:C
- removed C29: 0.1uF, symbol Device:C
- removed C51: C, symbol Device:C
- removed FB5: FerriteBead, Inductor_SMD:L_0805_2012Metric_Pad1.05x1.20mm_HandSolder, symbol Device:FerriteBead
- removed U7: REF35125QDBVRQ1, symbol Library:REF35125-Q1
- C23: renamed from C4; value C -> 0.1u
- U2: footprint VQFN-FCRLF22_RYF_TEX -> Footprint:VQFN-FCRLF22_RYF_TEX
- renumbered C5 to C22, C3 to C24, C2 to C25, C1 to C26, C6 to C27, C14 to C28, C16 to C29, C17 to C30, C15 to C31, C7 to C32, C13 to C33, C8 to C34, C12 to C35, R20 to R5, R21 to R6, R22 to R7, R23 to R8, R24 to R9
Other:
- note removed: "+1.25V Vref"
- note removed: "Ref for TLV6001"
- moved on the sheet: C27, J1, L1
