File: sensors.kicad_sch (KiCad schematic)
At the start: 23 parts, among them IC1 ACS724LMATR-20AB-T, IC2 ACS724LMATR-20AB-T, IC3 ACS724LMATR-20AB-T, U1 AMC1311QDWVRQ1, U6 MA732GQ-P

Commit message: CIPOS circuit
Parts:
- removed R5, R6: R, symbol Device:R
- added R12, R13: 10k, symbol Device:R
- added R14, R15: 4.99k, symbol Device:R
- added TP6, TP7: TestPoint, symbol Connector:TestPoint
- added U9: TLV6001DCK, Package_TO_SOT_SMD:SOT-353_SC-70-5, symbol Amplifier_Operational:TLV6001DCK
- C24: value 10nF -> 1uF
Connections:
- net GND: now also C24.2, U6.17 (PAD), U9.2 (V-)
- net Ib_sense: now reaches C19.1, IC3.12 (VIOUT)
- net Ib_sense: now also C22.1, IC2.12 (VIOUT)
- net at U1.6 (VOUTN): now also R12.1
- net +3.3V: now reaches C24.1
- net +3.3V: now also U6.13 (VDD), U9.5 (V+)
- net Ia_sense: now reaches C10.1, IC1.12 (VIOUT)
- net at U1.7 (VOUTP): now also R13.1
- net at U6.11 (MGL): now also TP6.1
- net at U6.16 (MGH): now also TP7.1
- net eQEPA: now reaches U6.2 (A)
- net eQEPZ: now reaches U6.3 (Z)
- net eQEPB: now reaches U6.6 (B)
- new net: R13.2, R14.1, U9.1 (+)
- new net: R12.2, R15.2, U9.3 (-)
- new net ADC1: R15.1, U9.4
- new net REFV: R14.2
- no-connect marks 6 -> 9
Other:
- note added: "0.1% resistors for exact gain"
- note added: "AMC1311 is used to measure the DC link voltage, this gives galvanic isolation."
- note added: "Current Sense"
- note added: "Data-Sheet"
- note added: "Data-sheet"
- note added: "Ref +1.25V for the TLV6001 is taken from the REF35125QDBVRQ1 TLV6001 is used to convert Differential out to single ended out put for the MCU,"
- note added: "Reference - Click Here"
- note added: "Supports upto 60,000RPM, Both axis and off axis Both SPI and eQEP supported"
- note added: "Voltage Sense"
- note removed: "Number of unit resistors depends on design requirements."
- moved on the sheet: C10, C11, C18, C19, C20, C21, C22, C23, C25, C26, C27, C9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

Commit message: #
Connections:
- net Ia_In renamed Iu_In
- net Ia_Out renamed Iu_Out
- net Ib_In renamed Iw_In
- net Ib_Out renamed Iw_Out
- net Ic_In renamed Iv_In
- net Ic_Out renamed Iv_Out
Other:
- note added: "Current Sensing 3phase"
- note added: "Inverter"
- note added: "M"
- note added: "Voltage sensing"
- moved on the sheet: C10, C11, C18, C19, C20, C21, C22, C23, C9, IC1, IC2, IC3

Commit message: #
Parts:
- added C52, C59: 1u, Capacitor_SMD:C_0805_2012Metric_Pad1.18x1.45mm_HandSolder, symbol Device:C
- added C53, C56, C58: 1n, Capacitor_SMD:C_0603_1608Metric_Pad1.08x0.95mm_HandSolder, symbol Device:C
- added C54, C55, C57: 100n, Capacitor_SMD:C_0603_1608Metric_Pad1.08x0.95mm_HandSolder, symbol Device:C
- added FB1, FB2: FerriteBead, Inductor_SMD:L_0805_2012Metric_Pad1.05x1.20mm_HandSolder, symbol Device:FerriteBead
- added IC6: AMC3311QDWERQ1, SOIC127P1030X265-16N, symbol AMC3311QDWERQ1:AMC3311QDWERQ1
- added IC7: OPA388QDBVRQ1, SOT95P280X145-5N, symbol OPA388QDBVRQ1:OPA388QDBVRQ1
- added R33, R61, R62, R63, R64, R66: 100k, Resistor_SMD:R_0603_1608Metric_Pad0.98x0.95mm_HandSolder, symbol Device:R
- added R34: 47k, Resistor_SMD:R_0603_1608Metric_Pad0.98x0.95mm_HandSolder, symbol Device:R
- added R51: 10k, Resistor_SMD:R_0603_1608Metric_Pad0.98x0.95mm_HandSolder, symbol Device:R
- added R52, R53: 150k, Resistor_SMD:R_0603_1608Metric_Pad0.98x0.95mm_HandSolder, symbol Device:R
- added R78: 2.2k, Resistor_SMD:R_0603_1608Metric_Pad0.98x0.95mm_HandSolder, symbol Device:R
- added TP13, TP14, TP15: TestPoint, symbol Connector:TestPoint
- added TP16, TP17: TestPoint, TestPoint:TestPoint_Keystone_5010-5014_Multipurpose, symbol Connector:TestPoint
- added TP18: TestPoint, TestPoint:TestPoint_Pad_1.0x1.0mm, symbol Connector:TestPoint
Connections:
- net +5V: now also C11.1, C18.1, C21.1, IC1.10 (VCC), IC2.10 (VCC), IC3.10 (VCC)
- net ADC1: now also TP15.1
- net GND: now also C58.1, C59.1, IC6.9 (GND), R33.2
- net GND1: now also TP14.1
- net at C25.1, R11.2, R9.1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: now also TP13.1
- new net: IC7.3 (+IN), R33.1, R63.1
- new net: R52.1, R62.2
- new net: C52.1, C53.1, C54.1, C55.1, C56.2, FB2.2, IC6.2 (DCDC_HGND), IC6.7 (HGND_1), IC6.8 (HGND_2), TP17.1
- new net: C52.2, C53.2, C54.2, IC6.1 (DCDC_OUT), IC6.3 (HLDO_IN)
- new net: FB1.1, R51.1, R52.2
- new net: FB1.2, IC6.6 (IN), TP16.1
- new net: IC7.1 (OUT), R64.2, R78.1
- new net: C55.2, C56.1, IC6.5 (HLDO_OUT)
- new net: R53.2, R61.1
- new net: FB2.1, R51.2, R53.1
- new net: IC7.4 (-IN), R64.1, R66.1
- new net: IC6.14 (DIAG), R34.2, TP18.1
- new net: C57.1, IC6.13 (LDO_OUT), IC6.16 (DCDC_IN)
- new net +3V3: IC7.5 (V+)
- new net +DCLink: R62.1
- new net -DCLink: R61.2
- new net 5V_DIG: C58.2, C59.2, IC6.12 (VDD), R34.1
- new net DC_OUTN: IC6.10 (OUTN), R66.2
- new net DC_OUTP: IC6.11 (OUTP), R63.2
- new net DC_Sense: R78.2
- new net GNDD: C57.2, IC6.15 (DCDC_GND), IC7.2 (V-)
Other:
- moved on the sheet: C11, C18, C21

Commit message: #
Parts:
- removed C10, C19, C22: (no value), symbol Device:C
- removed C25: 100pF, symbol Device:C
- removed C26: 100nF, symbol Device:C
- removed C27: 1uF, symbol Device:C
- removed R10, R11: R, symbol Device:R
- removed R12, R13: 10k, symbol Device:R
- removed R14, R15: 4.99k, symbol Device:R
- removed R9: RSNS, symbol Device:R
- removed TP13, TP14, TP15: TestPoint, symbol Connector:TestPoint
- removed U1: AMC1311QDWVRQ1, DWV8_TEX, symbol 2026-08-07_17-48-11:AMC1311QDWVRQ1
- removed U9: TLV6001DCK, Package_TO_SOT_SMD:SOT-353_SC-70-5, symbol Amplifier_Operational:TLV6001DCK
- added IC10, IC11, IC9: OPA388QDBVRQ1, Footprint:SOT95P280X145-5N, symbol OPA388QDBVRQ1:OPA388QDBVRQ1
- added R21, R24, R27: 10k, symbol Device:R
- added R22, R25, R28: 6.6k, symbol Device:R
- added R23, R26, R29: 100, symbol Device:R
- C11: value (none) -> 0.1uF
- C13: renamed from C21; value (none) -> 0.1u
- C15: renamed from C18; value (none) -> 0.1u
- IC1, IC2, IC3, IC6: footprint SOIC127P1030X265-16N -> Footprint:SOIC127P1030X265-16N
- IC7: footprint SOT95P280X145-5N -> Footprint:SOT95P280X145-5N
- R20: renamed from R78; value 2.2k -> 100
- renumbered C52 to C1, C9 to C10, C23 to C12, C20 to C14, C53 to C2, C54 to C3, C55 to C4, C56 to C5, C57 to C6, C58 to C7, C59 to C8, C24 to C9, R62 to R10, R52 to R11, R51 to R12, R53 to R13, R61 to R14, R34 to R15, R66 to R16, R63 to R17, R33 to R18, R64 to R19
Connections:
- net +3V3 is gone; now on net +3.3V: IC7.5 (V+)
- net GNDD is gone; now on net GND: C6.2, IC6.15 (DCDC_GND), IC7.2 (V-)
- net +3.3V: now also IC10.5 (V+), IC11.5 (V+), IC9.5 (V+)
- net +5V: now also R15.1
- net 5V_DIG: no longer R15.1
- net GND: now also IC10.2 (V-), IC11.2 (V-), IC9.2 (V-), R21.2, R24.2, R27.2
- net Ia_sense renamed Iu_out
- net Iu_out: now also IC9.3 (+IN)
- net Ib_sense renamed Iv_out
- net Iv_out: now also IC10.3 (+IN); no longer IC3.12 (VIOUT)
- net SPI3CLK renamed SPIACLK
- net SPI3CS renamed SPIACS
- net SPI3MISO renamed SPIAMISO
- net SPI3MOSI renamed SPIAMOSI
- new net: IC10.1 (OUT), R25.1, R26.2
- new net: IC10.4 (-IN), R24.1, R25.2
- new net: IC9.1 (OUT), R22.1, R23.2
- new net: IC9.4 (-IN), R21.1, R22.2
- new net: IC11.1 (OUT), R28.1, R29.2
- new net: IC11.4 (-IN), R27.1, R28.2
- new net ADC_IU: R23.1
- new net ADC_IV: R26.1
- new net ADC_IW: R29.1
- new net Iw_out: IC11.3 (+IN), IC3.12 (VIOUT)
Other:
- note removed: "0.1% resistors for exact gain"
- note removed: "AMC1311 is used to measure the DC link voltage, this gives galvanic isolation."
- note removed: "Ref +1.25V for the TLV6001 is taken from the REF35125QDBVRQ1 TLV6001 is used to convert Differential out to single ended out put for the MCU,"
- note removed: "Reference - Click Here"
- note removed: "Supports upto 60,000RPM, Both axis and off axis Both SPI and eQEP supported"
- note removed: "Voltage Sense"
- moved on the sheet: C1, C10, C12, C13, C14, C15, C2, C3, C4, C5, C6, C7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
